Commit message: sim: docu de lanzamiento (headless/GUI, modelo full/box, gotchas) + runs del dia
- COMO_LANZAR.md: lab.launch.py como paso 1 (headless default), eleccion de
  modelo G1_SIM_MODEL full/box con la fisica nueva (envolvente 0.44x1.10,
  puerta re-carvada 0.85-1.2 m), firma del doble-gzserver (exit 255 +
  'Entity already exists'), docker cp del URDF en la receta de instalacion
  (su ausencia causo el robot-fantasma del contenedor), y 3 sintomas nuevos
  en problemas tipicos.
- HANDOFF.md + g1_base.urdf (anti-vuelco): trabajo previo de la sesion.
- dataset + CSVs: runs sim del dia — 135307/141733/142356 (cuerpo fantasma,
  8-11 col), 165750/170306 (falso exito: vano 0.42), 175230 (9 col
  presionando el marco, sin JSON principal), 181212/182620/182859
  (VALIDACION: reached, 0 colisiones, 77-83 s).

Co-Authored-By: Claude Fable 5 <noreply@anthropic.com>

File: sim/g1_sim_pkg/urdf/g1_base.urdf (robot description, URDF)
Before this commit: robot g1_stand_in, 3 links, 2 joints
Links:
- link base_link: mass 20 -> 60
